Commit message: Improved URDF

File: src/description/fyp_bot1_description.urdf (robot description, URDF)
Before this commit: robot bot1/fyp_bot, 3 links, 2 joints
Links:
- added link bot1/middle_link; visual cylinder length=${base_thickness} radius=${base_radius}
- added link bot1/top_link; visual cylinder length=${base_thickness} radius=${base_radius}
Joints:
- added joint middle_joint: type fixed, parent bot1/base_link, child bot1/middle_link, origin xyz=0.0 0.0 ${spacer_height} rpy=0 0 0
- added joint top_joint: type fixed, parent bot1/middle_link, child bot1/top_link, origin xyz=0.0 0.0 ${spacer_height} rpy=0 0 0
- joint laser_joint: origin xyz=0.0 0.0 ${(base_thickness+(lidar_height/2))} rpy=0 0 0 -> xyz=0.0 0.0 ${((spacer_height*2)+base_thickness+(lidar_height/2))} rpy=0 0 0

File: src/description/fyp_bot2_description.urdf (robot description, URDF)
Before this commit: robot bot2/fyp_bot, 3 links, 2 joints
Links:
- added link bot2/middle_link; visual cylinder length=${base_thickness} radius=${base_radius}
- added link bot2/top_link; visual cylinder length=${base_thickness} radius=${base_radius}
Joints:
- added joint middle_joint: type fixed, parent bot2/base_link, child bot2/middle_link, origin xyz=0.0 0.0 ${spacer_height} rpy=0 0 0
- added joint top_joint: type fixed, parent bot2/middle_link, child bot2/top_link, origin xyz=0.0 0.0 ${spacer_height} rpy=0 0 0
- joint laser_joint: origin xyz=0.0 0.0 ${(base_thickness+(lidar_height/2))} rpy=0 0 0 -> xyz=0.0 0.0 ${((spacer_height*2)+base_thickness+(lidar_height/2))} rpy=0 0 0

File: src/description/fyp_bot_description.urdf (robot description, URDF)
Before this commit: robot fyp_bot, 4 links, 3 joints
Links:
- removed link imu_link
- added link middle_link; visual cylinder length=${base_thickness} radius=${base_radius}
- added link top_link; visual cylinder length=${base_thickness} radius=${base_radius}
Joints:
- removed joint imu_joint
- added joint middle_joint: type fixed, parent base_link, child middle_link, origin xyz=0.0 0.0 ${spacer_height} rpy=0 0 0
- added joint top_joint: type fixed, parent middle_link, child top_link, origin xyz=0.0 0.0 ${spacer_height} rpy=0 0 0
- joint laser_joint: origin xyz=0.0 0.0 ${(base_thickness+(lidar_height/2))} rpy=0 0 0 -> xyz=0.0 0.0 ${((spacer_height*2)+base_thickness+(lidar_height/2))} rpy=0 0 0
